File: Channel1Photodetect.sch (KiCad schematic (older format))
At the start: 11 parts, among them P201 CONN_01X01, U201 MCP6404, U202 LM339

Commit message: Start of connecting the layout
Parts:
- P201: value CONN_01X01 -> Sig1; ConradPN (none) -> Value; MPN (none) -> Value
Changed lines of the file:
@@
 P 6000 2350
 F 0 "P201" V 6100 2350 50  0000 C CNN
-F 1 "CONN_01X01" V 6100 2350 50  0001 C CNN
+F 1 "Sig1" V 6000 2150 50  0000 C CNN
 F 2 "Pin_Headers:Pin_Header_Straight_1x01" H 6000 2350 60  0001 C CNN
 F 3 "" H 6000 2350 60  0000 C CNN
+F 4 "Value" H 6000 2350 60  0001 C CNN "MPN"
+F 5 "Value" H 6000 2350 60  0001 C CNN "ConradPN"
 	1    6000 2350
 	0    -1   -1   0

Commit message: Completed the board layout
Parts:
- RV201: footprint DasBlinkInput:P090L-02F25BR10K -> DasBlinkInput:CT6EP; Link http://parts.io/detail/236178/P090L-02F25BR10K -> http://www.nidec-copal-electronics.com/e/catalog/trimmer/ct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; MPN P090L-02F25BR10K -> CT6EP103-ND
Connections:
- net labels added: PD1
- net labels removed: Channel1_Out
Changed lines of the file:
@@
 LIBS:memory
 LIBS:xilinx
-LIBS:special
 LIBS:microcontrollers
 LIBS:dsp
@@
 F 0 "RV201" H 5900 3800 50  0000 C CNN
 F 1 "POT" H 5900 3900 50  0000 C CNN
-F 2 "DasBlinkInput:P090L-02F25BR10K" H 5900 3900 60  0001 C CNN
+F 2 "DasBlinkInput:CT6EP" H 5900 3900 60  0001 C CNN
 F 3 "" H 5900 3900 60  0000 C CNN
-F 4 "P090L-02F25BR10K" H 5900 3900 60  0001 C CNN "MPN"
-F 5 "http://parts.io/detail/236178/P090L-02F25BR10K" H 5900 3900 60  0001 C CNN "Link"
+F 4 "CT6EP103-ND" H 5900 3900 60  0001 C CNN "MPN"
+F 5 "http://www.nidec-copal-electronics.com/e/catalog/trimmer/ct-6.pdf" H 5900 3900 60  0001 C CNN "Link"
 	1    5900 3900
 	0    1    1    0
@@
 	2650 3450 2650 3800
 Text HLabel 7900 2850 2    60   Input ~ 0
-Channel1_Out
+PD1
 Text HLabel 8050 4250 2    60   Input ~ 0
 REF_OUT

Commit message: Updated the schematic for the BOM and generated the BOM
Parts:
- PD201: ConradPN (none) -> N/A; MPN VBPW34SR -> VBPW34FAS
- R201: ConradPN (none) -> 1209000 - 62
- RV201: ConradPN (none) -> N/A; MPN CT6EP103-ND -> CT6EP103
- U201: ConradPN (none) -> 1084976 - 62
- U202: ConradPN (none) -> 1010753 - 62
Changed lines of the file:
@@
 F 4 "RC1206FR-071ML" H 4550 1900 60  0001 C CNN "MPN"
 F 5 "http://parts.io/detail/880921/RC1206FR-071ML" H 4550 1900 60  0001 C CNN "Link"
+F 6 "1209000 - 62" V 4550 1900 60  0001 C CNN "ConradPN"
 	1    4550 1900
 	0    1    1    0
@@
 F 4 "MCP6404-E/SL" H 4600 2750 60  0001 C CNN "MPN"
 F 5 "http://parts.io/detail/3584122/MCP6404-E%2FSL" H 4600 2750 60  0001 C CNN "Link"
+F 6 "1084976 - 62" H 4600 2750 60  0001 C CNN "ConradPN"
 	1    4600 2750
 	1    0    0    1
@@
 F 2 "DasBlinkInput:VBPW34SR*" V 2650 3350 60  0001 C CNN
 F 3 "" V 2650 3350 60  0000 C CNN
-F 4 "VBPW34SR" H 2650 3350 60  0001 C CNN "MPN"
+F 4 "VBPW34FAS" H 2650 3350 60  0001 C CNN "MPN"
 F 5 "http://parts.io/detail/100078259/VBPW34SR" H 2650 3350 60  0001 C CNN "Link"
+F 6 "N/A" H 2650 3350 60  0001 C CNN "ConradPN"
 	1    2650 3350
 	0    -1   -1   0
@@
 F 4 "LM339DE4" H 7100 2850 60  0001 C CNN "MPN"
 F 5 "http://parts.io/detail/916254/LM339DE4" H 7100 2850 60  0001 C CNN "Link"
+F 6 "1010753 - 62 " H 7100 2850 60  0001 C CNN "ConradPN"
 	1    7100 2850
 	1    0    0    -1
@@
 F 2 "DasBlinkInput:CT6EP" H 5900 3900 60  0001 C CNN
 F 3 "" H 5900 3900 60  0000 C CNN
-F 4 "CT6EP103-ND" H 5900 3900 60  0001 C CNN "MPN"
+F 4 "CT6EP103" H 5900 3900 60  0001 C CNN "MPN"
 F 5 "http://www.nidec-copal-electronics.com/e/catalog/trimmer/ct-6.pdf" H 5900 3900 60  0001 C CNN "Link"
+F 6 "N/A" H 5900 3900 60  0001 C CNN "ConradPN"
 	1    5900 3900
 	0    1    1    0

Commit message: Changes to the BOM
Parts:
- PD201: ConradPN N/A -> 152965 - 62
- RV201: ConradPN N/A -> 675101 - 62
Changed lines of the file:
@@
 F 3 "" V 2650 3350 60  0000 C CNN
 F 4 "VBPW34FAS" H 2650 3350 60  0001 C CNN "MPN"
-F 5 "http://parts.io/detail/100078259/VBPW34SR" H 2650 3350 60  0001 C CNN "Link"
-F 6 "N/A" H 2650 3350 60  0001 C CNN "ConradPN"
+F 5 "152965 - 62" H 2650 3350 60  0001 C CNN "ConradPN"
+F 6 "http://parts.io/detail/100078259/VBPW34SR" H 2650 3350 60  0001 C CNN "Link"
 	1    2650 3350
 	0    -1   -1   0
@@
 F 3 "" H 5900 3900 60  0000 C CNN
 F 4 "CT6EP103" H 5900 3900 60  0001 C CNN "MPN"
-F 5 "http://www.nidec-copal-electronics.com/e/catalog/trimmer/ct-6.pdf" H 5900 3900 60  0001 C CNN "Link"
-F 6 "N/A" H 5900 3900 60  0001 C CNN "ConradPN"
+F 5 "675101 - 62" H 5900 3900 60  0001 C CNN "ConradPN"
+F 6 "http://www.nidec-copal-electronics.com/e/catalog/trimmer/ct-6.pdf" H 5900 3900 60  0001 C CNN "Link"
 	1    5900 3900
 	0    1    1    0

Commit message: Checkin before moving to Vagrant
Parts:
- R203: value 10K -> 0
- RV201: value POT -> 10K
Connections:
- wire segments 37 -> 47
Changed lines of the file:
@@
 LIBS:valves
 LIBS:DasBlinkInput
-LIBS:DasBlinkInput-cache
 EELAYER 25 0
 EELAYER END
@@
 $EndComp
 Wire Wire Line
-	5100 2750 6750 2750
+	5100 2750 5550 2750
+Wire Wire Line
+	5550 2750 6000 2750
+Wire Wire Line
+	6000 2750 6750 2750
 Wire Wire Line
 	5550 1900 5550 2750
 Wire Wire Line
-	4700 1900 5550 1900
+	4700 1900 4950 1900
+Wire Wire Line
+	4950 1900 5550 1900
 Wire Wire Line
 	4100 2650 2650 2650
 Wire Wire Line
-	2650 1900 2650 3250
-Wire Wire Line
-	2650 1900 4400 1900
+	2650 1900 2650 2650
+Wire Wire Line
+	2650 2650 2650 3250
+Wire Wire Line
+	2650 1900 4200 1900
+Wire Wire Line
+	4200 1900 4400 1900
 Connection ~ 2650 2650
 Wire Wire Line
@@
 	4500 3150 4500 3400
 Wire Wire Line
-	4150 3400 4750 3400
+	4150 3400 4500 3400
+Wire Wire Line
+	4500 3400 4750 3400
 $Comp
 L C C202
@@
 P 6250 3400
 F 0 "R203" V 6330 3400 50  0000 C CNN
-F 1 "10K" V 6250 3400 50  0000 C CNN
+F 1 "0" V 6250 3400 50  0000 C CNN
 F 2 "Resistors_SMD:R_0805_HandSoldering" V 6180 3400 30  0001 C CNN
 F 3 "" H 6250 3400 30  0000 C CNN
@@
 P 5900 3900
 F 0 "RV201" H 5900 3800 50  0000 C CNN
-F 1 "POT" H 5900 3900 50  0000 C CNN
+F 1 "10K" H 5900 3900 50  0000 C CNN
 F 2 "DasBlinkInput:CT6EP" H 5900 3900 60  0001 C CNN
 F 3 "" H 5900 3900 60  0000 C CNN
@@
 	6250 3900 6050 3900
 Wire Wire Line
-	5900 4150 5900 4400
-Wire Wire Line
-	5900 4250 8050 4250
+	5900 4150 5900 4250
+Wire Wire Line
+	5900 4250 5900 4400
+Wire Wire Line
+	5900 4250 6550 4250
+Wire Wire Line
+	6550 4250 8050 4250
 Wire Wire Line
 	6550 4250 6550 2950
@@
 Connection ~ 5900 4250
 Wire Wire Line
-	7450 2850 7900 2850
+	7450 2850 8100 2850
 Text GLabel 6550 2150 0    60   Input ~ 0
 3V
 Wire Wire Line
-	6550 2150 7150 2150
+	6550 2150 7000 2150
+Wire Wire Line
+	7000 2150 7150 2150
 $Comp
 L C C203
@@
 Wire Wire Line
 	2650 3450 2650 3800
-Text HLabel 7900 2850 2    60   Input ~ 0
+Text HLabel 8100 2850 2    60   Input ~ 0
 PD1
 Text HLabel 8050 4250 2    60   Input ~ 0
@@
 VGND
 Wire Wire Line
-	2400 3800 3600 3800
+	2400 3800 2650 3800
+Wire Wire Line
+	2650 3800 3600 3800
 Wire Wire Line
 	3600 3800 3600 2850

Commit message: Clean up and correctsion to the layout. Added the pull up resistors
Parts:
- C201, C202, C203: footprint Capacitors_SMD:C_0805_HandSoldering -> Capacitors_SMD:C_0805
- R202, R203: footprint Resistors_SMD:R_0805_HandSoldering -> Resistors_SMD:R_0805
Connections:
- wire segments 47 -> 37
Changed lines of the file:
@@
 LIBS:valves
 LIBS:DasBlinkInput
+LIBS:DasBlinkInput-cache
 EELAYER 25 0
 EELAYER END
@@
 F 0 "C201" H 4625 1600 50  0000 L CNN
 F 1 "100p" H 4625 1400 50  0000 L CNN
-F 2 "Capacitors_SMD:C_0805_HandSoldering" H 4638 1350 30  0001 C CNN
+F 2 "Capacitors_SMD:C_0805" H 4638 1350 30  0001 C CNN
 F 3 "" H 4600 1500 60  0000 C CNN
 	1    4600 1500
@@
 $EndComp
 Wire Wire Line
-	5100 2750 5550 2750
-Wire Wire Line
-	5550 2750 6000 2750
-Wire Wire Line
-	6000 2750 6750 2750
+	5100 2750 6800 2750
 Wire Wire Line
 	5550 1900 5550 2750
 Wire Wire Line
-	4700 1900 4950 1900
-Wire Wire Line
-	4950 1900 5550 1900
+	4700 1900 5550 1900
 Wire Wire Line
 	4100 2650 2650 2650
 Wire Wire Line
-	2650 1900 2650 2650
-Wire Wire Line
-	2650 2650 2650 3250
-Wire Wire Line
-	2650 1900 4200 1900
-Wire Wire Line
-	4200 1900 4400 1900
+	2650 1900 2650 3250
+Wire Wire Line
+	2650 1900 4400 1900
 Connection ~ 2650 2650
 Wire Wire Line
@@
 	4500 3150 4500 3400
 Wire Wire Line
-	4150 3400 4500 3400
-Wire Wire Line
-	4500 3400 4750 3400
+	4150 3400 4750 3400
 $Comp
 L C C202
@@
 F 0 "C202" H 4925 3500 50  0000 L CNN
 F 1 "0.1U" H 4925 3300 50  0000 L CNN
-F 2 "Capacitors_SMD:C_0805_HandSoldering" H 4938 3250 30  0001 C CNN
+F 2 "Capacitors_SMD:C_0805" H 4938 3250 30  0001 C CNN
 F 3 "" H 4900 3400 60  0000 C CNN
 	1    4900 3400
@@
 F 0 "R203" V 6330 3400 50  0000 C CNN
 F 1 "0" V 6250 3400 50  0000 C CNN
-F 2 "Resistors_SMD:R_0805_HandSoldering" V 6180 3400 30  0001 C CNN
+F 2 "Resistors_SMD:R_0805" V 6180 3400 30  0001 C CNN
 F 3 "" H 6250 3400 30  0000 C CNN
 	1    6250 3400
@@
 F 0 "R202" V 5980 4550 50  0000 C CNN
 F 1 "10K" V 5900 4550 50  0000 C CNN
-F 2 "Resistors_SMD:R_0805_HandSoldering" V 5830 4550 30  0001 C CNN
+F 2 "Resistors_SMD:R_0805" V 5830 4550 30  0001 C CNN
 F 3 "" H 5900 4550 30  0000 C CNN
 	1    5900 4550
@@
 	6250 3900 6050 3900
 Wire Wire Line
-	5900 4150 5900 4250
-Wire Wire Line
-	5900 4250 5900 4400
-Wire Wire Line
-	5900 4250 6550 4250
-Wire Wire Line
-	6550 4250 8050 4250
+	5900 4150 5900 4400
+Wire Wire Line
+	5900 4250 8050 4250
 Wire Wire Line
 	6550 4250 6550 2950
 Wire Wire Line
-	6550 2950 6750 2950
+	6550 2950 6800 2950
 Connection ~ 5900 4250
 Wire Wire Line
-	7450 2850 8100 2850
+	7400 2850 8100 2850
 Text GLabel 6550 2150 0    60   Input ~ 0
 3V
 Wire Wire Line
-	6550 2150 7000 2150
-Wire Wire Line
-	7000 2150 7150 2150
+	6550 2150 7150 2150
 $Comp
 L C C203
@@
 F 0 "C203" H 7325 2250 50  0000 L CNN
 F 1 "0.1U" H 7325 2050 50  0000 L CNN
-F 2 "Capacitors_SMD:C_0805_HandSoldering" H 7338 2000 30  0001 C CNN
+F 2 "Capacitors_SMD:C_0805" H 7338 2000 30  0001 C CNN
 F 3 "" H 7300 2150 60  0000 C CNN
 	1    7300 2150
@@
 VGND
 Wire Wire Line
-	2400 3800 2650 3800
-Wire Wire Line
-	2650 3800 3600 3800
+	2400 3800 3600 3800
 Wire Wire Line
 	3600 3800 3600 2850
