File: Channel2Photodetect.sch (KiCad schematic (older format))
At the start: 6 parts, among them P301 CONN_01X01, U201 MCP6404, U202 LM339

Commit message: Start of connecting the layout
Parts:
- P301: value CONN_01X01 -> Sig2; ConradPN (none) -> Value; MPN (none) -> Value
Changed lines of the file:
@@
 P 6400 2550
 F 0 "P301" H 6400 2650 50  0000 C CNN
-F 1 "CONN_01X01" V 6500 2550 50  0000 C CNN
+F 1 "Sig2" V 6400 2400 50  0000 C CNN
 F 2 "Pin_Headers:Pin_Header_Straight_1x01" H 6400 2550 60  0001 C CNN
 F 3 "" H 6400 2550 60  0000 C CNN
+F 4 "Value" H 6400 2550 60  0001 C CNN "MPN"
+F 5 "Value" H 6400 2550 60  0001 C CNN "ConradPN"
 	1    6400 2550
 	0    -1   -1   0

Commit message: Completed the board layout
Connections:
- net labels added: PD2
- net labels removed: Channel2_Out
Changed lines of the file:
@@
 LIBS:memory
 LIBS:xilinx
-LIBS:special
 LIBS:microcontrollers
 LIBS:dsp
@@
 	7800 3100 8250 3100
 Text HLabel 8250 3100 2    60   Input ~ 0
-Channel2_Out
+PD2
 Text HLabel 8400 4500 2    60   Input ~ 0
 REF_IN

Commit message: Updated the schematic for the BOM and generated the BOM
Parts:
- PD301: ConradPN (none) -> N/A; MPN VBPW34SR -> VBPW34FAS
- R301: ConradPN (none) -> 1209000 - 62
- U201: ConradPN (none) -> 1084976 - 62
- U202: ConradPN (none) -> 1010753 - 62
Changed lines of the file:
@@
 F 4 "RC1206FR-071ML" H 4900 2150 60  0001 C CNN "MPN"
 F 5 "http://parts.io/detail/880921/RC1206FR-071ML" H 4900 2150 60  0001 C CNN "Link"
+F 6 "1209000 - 62" H 4900 2150 60  0001 C CNN "ConradPN"
 	1    4900 2150
 	0    1    1    0
@@
 F 4 "MCP6404-E/SL" H 4950 3000 60  0001 C CNN "MPN"
 F 5 "http://parts.io/detail/3584122/MCP6404-E%2FSL" H 4950 3000 60  0001 C CNN "Link"
+F 6 "1084976 - 62" H 4950 3000 60  0001 C CNN "ConradPN"
 	2    4950 3000
 	1    0    0    1
@@
 F 2 "DasBlinkInput:VBPW34SR*" V 3550 3600 60  0001 C CNN
 F 3 "" V 3550 3600 60  0000 C CNN
-F 4 "VBPW34SR" H 3550 3600 60  0001 C CNN "MPN"
+F 4 "VBPW34FAS" H 3550 3600 60  0001 C CNN "MPN"
 F 5 "http://parts.io/detail/100078259/VBPW34SR" H 3550 3600 60  0001 C CNN "Link"
+F 6 "N/A" H 3550 3600 60  0001 C CNN "ConradPN"
 	1    3550 3600
 	0    -1   -1   0
@@
 F 4 "LM339DE4" H 7450 3100 60  0001 C CNN "MPN"
 F 5 "http://parts.io/detail/916254/LM339DE4" H 7450 3100 60  0001 C CNN "Link"
+F 6 "1010753 - 62 " H 7450 3100 60  0001 C CNN "ConradPN"
 	2    7450 3100
 	1    0    0    -1

Commit message: Changes to the BOM
Parts:
- PD301: ConradPN N/A -> 152965 - 62
Changed lines of the file:
@@
 F 3 "" V 3550 3600 60  0000 C CNN
 F 4 "VBPW34FAS" H 3550 3600 60  0001 C CNN "MPN"
-F 5 "http://parts.io/detail/100078259/VBPW34SR" H 3550 3600 60  0001 C CNN "Link"
-F 6 "N/A" H 3550 3600 60  0001 C CNN "ConradPN"
+F 5 "152965 - 62" H 3550 3600 60  0001 C CNN "ConradPN"
+F 6 "http://parts.io/detail/100078259/VBPW34SR" H 3550 3600 60  0001 C CNN "Link"
 	1    3550 3600
 	0    -1   -1   0

Commit message: Clean up and correctsion to the layout. Added the pull up resistors
Parts:
- C301: footprint Capacitors_SMD:C_0805_HandSoldering -> Capacitors_SMD:C_0805
Changed lines of the file:
@@
 LIBS:valves
 LIBS:DasBlinkInput
+LIBS:DasBlinkInput-cache
 EELAYER 25 0
 EELAYER END
@@
 F 0 "C301" H 4975 1850 50  0000 L CNN
 F 1 "100p" H 4975 1650 50  0000 L CNN
-F 2 "Capacitors_SMD:C_0805_HandSoldering" H 4988 1600 30  0001 C CNN
+F 2 "Capacitors_SMD:C_0805" H 4988 1600 30  0001 C CNN
 F 3 "" H 4950 1750 60  0000 C CNN
 	1    4950 1750
@@
 $EndComp
 Wire Wire Line
-	5450 3000 7100 3000
+	5450 3000 7150 3000
 Wire Wire Line
 	5900 2150 5900 3000
@@
 	6900 4500 6900 3200
 Wire Wire Line
-	6900 3200 7100 3200
+	6900 3200 7150 3200
 Wire Wire Line
-	7800 3100 8250 3100
+	7750 3100 8250 3100
 Text HLabel 8250 3100 2    60   Input ~ 0
 PD2
