File: Channel3PhotoDetect.sch (KiCad schematic (older format))
At the start: 6 parts, among them P401 CONN_01X01, U201 MCP6404, U202 LM339

Commit message: Start of connecting the layout
Parts:
- P401: value CONN_01X01 -> Sig3
Changed lines of the file:
@@
 P 6550 2400
 F 0 "P401" H 6550 2500 50  0000 C CNN
-F 1 "CONN_01X01" V 6650 2400 50  0000 C CNN
+F 1 "Sig3" V 6550 2250 50  0000 C CNN
 F 2 "Pin_Headers:Pin_Header_Straight_1x01" H 6550 2400 60  0001 C CNN
 F 3 "" H 6550 2400 60  0000 C CNN

Commit message: Completed the board layout
Connections:
- net labels added: PD3
- net labels removed: Channel3_Out
Changed lines of the file:
@@
 LIBS:memory
 LIBS:xilinx
-LIBS:special
 LIBS:microcontrollers
 LIBS:dsp
@@
 	7900 2900 8350 2900
 Text HLabel 8350 2900 2    60   Input ~ 0
-Channel3_Out
+PD3
 Text HLabel 8500 4300 2    60   Input ~ 0
 REF_IN

Commit message: Updated the schematic for the BOM and generated the BOM
Parts:
- PD401: ConradPN (none) -> N/A; MPN VBPW34SR -> VBPW34FAS
- R401: ConradPN (none) -> 1209000 - 62
- U201: ConradPN (none) -> 1084976 - 62
- U202: ConradPN (none) -> 1010753 - 62
Changed lines of the file:
@@
 F 4 "RC1206FR-071ML" H 5000 1950 60  0001 C CNN "MPN"
 F 5 "http://parts.io/detail/880921/RC1206FR-071ML" H 5000 1950 60  0001 C CNN "Link"
+F 6 "1209000 - 62" H 5000 1950 60  0001 C CNN "ConradPN"
 	1    5000 1950
 	0    1    1    0
@@
 F 4 "MCP6404-E/SL" H 5050 2800 60  0001 C CNN "MPN"
 F 5 "http://parts.io/detail/3584122/MCP6404-E%2FSL" H 5050 2800 60  0001 C CNN "Link"
+F 6 "1084976 - 62" H 5050 2800 60  0001 C CNN "ConradPN"
 	3    5050 2800
 	1    0    0    1
@@
 F 2 "DasBlinkInput:VBPW34SR*" V 3650 3400 60  0001 C CNN
 F 3 "" V 3650 3400 60  0000 C CNN
-F 4 "VBPW34SR" H 3650 3400 60  0001 C CNN "MPN"
+F 4 "VBPW34FAS" H 3650 3400 60  0001 C CNN "MPN"
 F 5 "http://parts.io/detail/100078259/VBPW34SR" H 3650 3400 60  0001 C CNN "Link"
+F 6 "N/A" H 3650 3400 60  0001 C CNN "ConradPN"
 	1    3650 3400
 	0    -1   -1   0
@@
 F 4 "LM339DE4" H 7550 2900 60  0001 C CNN "MPN"
 F 5 "http://parts.io/detail/916254/LM339DE4" H 7550 2900 60  0001 C CNN "Link"
+F 6 "1010753 - 62 " H 7550 2900 60  0001 C CNN "ConradPN"
 	3    7550 2900
 	1    0    0    -1

Commit message: Changes to the BOM
Parts:
- PD401: ConradPN N/A -> 152965 - 62
Changed lines of the file:
@@
 F 3 "" V 3650 3400 60  0000 C CNN
 F 4 "VBPW34FAS" H 3650 3400 60  0001 C CNN "MPN"
-F 5 "http://parts.io/detail/100078259/VBPW34SR" H 3650 3400 60  0001 C CNN "Link"
-F 6 "N/A" H 3650 3400 60  0001 C CNN "ConradPN"
+F 5 "152965 - 62" H 3650 3400 60  0001 C CNN "ConradPN"
+F 6 "http://parts.io/detail/100078259/VBPW34SR" H 3650 3400 60  0001 C CNN "Link"
 	1    3650 3400
 	0    -1   -1   0

Commit message: Clean up and correctsion to the layout. Added the pull up resistors
Parts:
- C401: footprint Capacitors_SMD:C_0805_HandSoldering -> Capacitors_SMD:C_0805
Changed lines of the file:
@@
 LIBS:valves
 LIBS:DasBlinkInput
+LIBS:DasBlinkInput-cache
 EELAYER 25 0
 EELAYER END
@@
 F 0 "C401" H 5075 1650 50  0000 L CNN
 F 1 "100p" H 5075 1450 50  0000 L CNN
-F 2 "Capacitors_SMD:C_0805_HandSoldering" H 5088 1400 30  0001 C CNN
+F 2 "Capacitors_SMD:C_0805" H 5088 1400 30  0001 C CNN
 F 3 "" H 5050 1550 60  0000 C CNN
 	1    5050 1550
@@
 $EndComp
 Wire Wire Line
-	5550 2800 7200 2800
+	5550 2800 7250 2800
 Wire Wire Line
 	6000 1950 6000 2800
@@
 	7000 4300 7000 3000
 Wire Wire Line
-	7000 3000 7200 3000
+	7000 3000 7250 3000
 Wire Wire Line
-	7900 2900 8350 2900
+	7850 2900 8350 2900
 Text HLabel 8350 2900 2    60   Input ~ 0
 PD3
