File: Channel4PhotoDetect.sch (KiCad schematic (older format))
At the start: 6 parts, among them P501 CONN_01X01, U201 MCP6404, U202 LM339

Commit message: Start of connecting the layout
Parts:
- P501: value CONN_01X01 -> Sig4
Changed lines of the file:
@@
 P 6450 2400
 F 0 "P501" H 6450 2500 50  0000 C CNN
-F 1 "CONN_01X01" V 6550 2400 50  0000 C CNN
+F 1 "Sig4" V 6450 2250 50  0000 C CNN
 F 2 "Pin_Headers:Pin_Header_Straight_1x01" H 6450 2400 60  0001 C CNN
 F 3 "" H 6450 2400 60  0000 C CNN

Commit message: Completed the board layout
Connections:
- net labels added: PD4
- net labels removed: Channel4_Out
Changed lines of the file:
@@
 LIBS:memory
 LIBS:xilinx
-LIBS:special
 LIBS:microcontrollers
 LIBS:dsp
@@
 	3250 3600 3250 3950
 Text HLabel 8250 3000 2    60   Input ~ 0
-Channel4_Out
+PD4
 Text HLabel 8400 4400 2    60   Input ~ 0
 REF_IN

Commit message: Updated the schematic for the BOM and generated the BOM
Parts:
- PD501: ConradPN (none) -> N/A; MPN VBPW34SR -> VBPW34FAS
- R501: ConradPN (none) -> 1209000 - 62
- U201: ConradPN (none) -> 1084976 - 62
- U202: ConradPN (none) -> 1010753 - 62
Changed lines of the file:
@@
 F 4 "RC1206FR-071ML" H 4900 2050 60  0001 C CNN "MPN"
 F 5 "http://parts.io/detail/880921/RC1206FR-071ML" H 4900 2050 60  0001 C CNN "Link"
+F 6 "1209000 - 62" H 4900 2050 60  0001 C CNN "ConradPN"
 	1    4900 2050
 	0    1    1    0
@@
 F 4 "MCP6404-E/SL" H 4950 2900 60  0001 C CNN "MPN"
 F 5 "http://parts.io/detail/3584122/MCP6404-E%2FSL" H 4950 2900 60  0001 C CNN "Link"
+F 6 "1084976 - 62" H 4950 2900 60  0001 C CNN "ConradPN"
 	4    4950 2900
 	1    0    0    1
@@
 F 2 "DasBlinkInput:VBPW34SR*" V 3250 3500 60  0001 C CNN
 F 3 "" V 3250 3500 60  0000 C CNN
-F 4 "VBPW34SR" H 3250 3500 60  0001 C CNN "MPN"
+F 4 "VBPW34FAS" H 3250 3500 60  0001 C CNN "MPN"
 F 5 "http://parts.io/detail/100078259/VBPW34SR" H 3250 3500 60  0001 C CNN "Link"
+F 6 "N/A" H 3250 3500 60  0001 C CNN "ConradPN"
 	1    3250 3500
 	0    -1   -1   0
@@
 F 4 "LM339DE4" H 7450 3000 60  0001 C CNN "MPN"
 F 5 "http://parts.io/detail/916254/LM339DE4" H 7450 3000 60  0001 C CNN "Link"
+F 6 "1010753 - 62 " H 7450 3000 60  0001 C CNN "ConradPN"
 	4    7450 3000
 	1    0    0    -1

Commit message: Changes to the BOM
Parts:
- PD501: ConradPN N/A -> 152965 - 62
Changed lines of the file:
@@
 F 3 "" V 3250 3500 60  0000 C CNN
 F 4 "VBPW34FAS" H 3250 3500 60  0001 C CNN "MPN"
-F 5 "http://parts.io/detail/100078259/VBPW34SR" H 3250 3500 60  0001 C CNN "Link"
-F 6 "N/A" H 3250 3500 60  0001 C CNN "ConradPN"
+F 5 "152965 - 62" H 3250 3500 60  0001 C CNN "ConradPN"
+F 6 "http://parts.io/detail/100078259/VBPW34SR" H 3250 3500 60  0001 C CNN "Link"
 	1    3250 3500
 	0    -1   -1   0

Commit message: Clean up and correctsion to the layout. Added the pull up resistors
Parts:
- C501: footprint Capacitors_SMD:C_0805_HandSoldering -> Capacitors_SMD:C_0805
Changed lines of the file:
@@
 LIBS:valves
 LIBS:DasBlinkInput
+LIBS:DasBlinkInput-cache
 EELAYER 25 0
 EELAYER END
@@
 F 0 "C501" H 4975 1750 50  0000 L CNN
 F 1 "100p" H 4975 1550 50  0000 L CNN
-F 2 "Capacitors_SMD:C_0805_HandSoldering" H 4988 1500 30  0001 C CNN
+F 2 "Capacitors_SMD:C_0805" H 4988 1500 30  0001 C CNN
 F 3 "" H 4950 1650 60  0000 C CNN
 	1    4950 1650
@@
 $EndComp
 Wire Wire Line
-	5450 2900 7100 2900
+	5450 2900 7150 2900
 Wire Wire Line
 	5900 2050 5900 2900
@@
 	6900 4400 6900 3100
 Wire Wire Line
-	6900 3100 7100 3100
+	6900 3100 7150 3100
 Wire Wire Line
-	7800 3000 8250 3000
+	7750 3000 8250 3000
 Wire Wire Line
 	3250 3600 3250 3950
