File: DasBlinkInput.sch (KiCad schematic (older format))
At the start: 11 parts, among them P101 CONN_01X02, P102 CONN_01X01, P103 CONN_01X01, P104 CONN_01X01, P105 CONN_01X05, U101 LP2980IM5-3.0/NOPB

Commit message: Start of connecting the layout
Parts:
- P101: value CONN_01X02 -> Vin; ConradPN (none) -> Value; MPN (none) -> Value
- P102: value CONN_01X01 -> VGND; ConradPN (none) -> Value; MPN (none) -> Value
- P103: value CONN_01X01 -> 3V; ConradPN (none) -> Value; MPN (none) -> Value
- P104: value CONN_01X01 -> GND; ConradPN (none) -> Value; MPN (none) -> Value
- P105: value CONN_01X05 -> Output; ConradPN (none) -> Value; MPN (none) -> Value
Changed lines of the file:
@@
 P 8650 1800
 F 0 "P105" H 8650 2100 50  0000 C CNN
-F 1 "CONN_01X05" V 8750 1800 50  0001 C CNN
+F 1 "Output" V 8750 1800 50  0000 C CNN
 F 2 "Pin_Headers:Pin_Header_Straight_1x05" H 8650 1800 60  0001 C CNN
 F 3 "" H 8650 1800 60  0000 C CNN
+F 4 "Value" H 8650 1800 60  0001 C CNN "MPN"
+F 5 "Value" H 8650 1800 60  0001 C CNN "ConradPN"
 	1    8650 1800
 	1    0    0    -1
@@
 P 950 1600
 F 0 "P101" H 950 1750 50  0000 C CNN
-F 1 "CONN_01X02" V 1050 1600 50  0001 C CNN
+F 1 "Vin" H 950 1400 50  0000 C CNN
 F 2 "Pin_Headers:Pin_Header_Straight_1x02" H 950 1600 60  0001 C CNN
 F 3 "" H 950 1600 60  0000 C CNN
+F 4 "Value" H 950 1600 60  0001 C CNN "MPN"
+F 5 "Value" H 950 1600 60  0001 C CNN "ConradPN"
 	1    950  1600
 	-1   0    0    1
@@
 P 4400 1200
 F 0 "P103" V 4500 1200 50  0000 C CNN
-F 1 "CONN_01X01" V 4500 1200 50  0001 C CNN
+F 1 "3V" V 4400 1100 50  0000 C CNN
 F 2 "Pin_Headers:Pin_Header_Straight_1x01" H 4400 1200 60  0001 C CNN
 F 3 "" H 4400 1200 60  0000 C CNN
+F 4 "Value" H 4400 1200 60  0001 C CNN "MPN"
+F 5 "Value" H 4400 1200 60  0001 C CNN "ConradPN"
 	1    4400 1200
 	0    -1   -1   0
@@
 P 1750 3650
 F 0 "P102" V 1850 3650 50  0000 C CNN
-F 1 "CONN_01X01" V 1850 3650 50  0001 C CNN
+F 1 "VGND" V 1750 3450 50  0000 C CNN
 F 2 "Pin_Headers:Pin_Header_Straight_1x01" H 1750 3650 60  0001 C CNN
 F 3 "" H 1750 3650 60  0000 C CNN
+F 4 "Value" H 1750 3650 60  0001 C CNN "MPN"
+F 5 "Value" H 1750 3650 60  0001 C CNN "ConradPN"
 	1    1750 3650
 	0    -1   -1   0
@@
 P 4400 3400
 F 0 "P104" V 4550 3400 50  0000 C CNN
-F 1 "CONN_01X01" V 4500 3400 50  0001 C CNN
+F 1 "GND" V 4400 3550 50  0000 C CNN
 F 2 "Pin_Headers:Pin_Header_Straight_1x01" H 4400 3400 60  0001 C CNN
 F 3 "" H 4400 3400 60  0000 C CNN
+F 4 "Value" H 4400 3400 60  0001 C CNN "MPN"
+F 5 "Value" H 4400 3400 60  0001 C CNN "ConradPN"
 	1    4400 3400
 	0    1    1    0

Commit message: Completed the board layout
Parts:
- added P106: Vref, Pin_Headers:Pin_Header_Straight_1x01, symbol CONN_01X01
Connections:
- wire segments 36 -> 37
Changed lines of the file:
@@
 LIBS:memory
 LIBS:xilinx
-LIBS:special
 LIBS:microcontrollers
 LIBS:dsp
@@
 F0 "Channel 1 Photodetect" 60
 F1 "Channel1Photodetect.sch" 60
-F2 "Channel1_Out" I R 6700 1600 60
+F2 "PD1" I R 6700 1600 60
 F3 "REF_OUT" I L 5850 1950 60
 $EndSheet
@@
 F0 "Channel 2 Photodetect" 60
 F1 "Channel2Photodetect.sch" 60
-F2 "Channel2_Out" I R 6700 2900 60
+F2 "PD2" I R 6700 2900 60
 F3 "REF_IN" I L 5850 3200 60
 $EndSheet
@@
 F0 "Channel 3 PhotoDetect" 60
 F1 "Channel3PhotoDetect.sch" 60
-F2 "Channel3_Out" I R 6700 4050 60
+F2 "PD3" I R 6700 4050 60
 F3 "REF_IN" I L 5850 4450 60
 $EndSheet
@@
 F0 "Channel 4 PhotoDetect" 60
 F1 "Channel4PhotoDetect.sch" 60
-F2 "Channel4_Out" I R 6750 5250 60
+F2 "PD4" I R 6750 5250 60
 F3 "REF_IN" I L 5850 5600 60
 $EndSheet
@@
 $EndComp
 Connection ~ 4400 3050
+$Comp
+L CONN_01X01 P106
+U 1 1 55657041
+P 5100 3750
+F 0 "P106" V 5200 3750 50  0000 C CNN
+F 1 "Vref" V 5100 3550 50  0000 C CNN
+F 2 "Pin_Headers:Pin_Header_Straight_1x01" H 5100 3750 60  0001 C CNN
+F 3 "" H 5100 3750 60  0000 C CNN
+F 4 "Value" H 5100 3750 60  0001 C CNN "MPN"
+F 5 "Value" H 5100 3750 60  0001 C CNN "Link"
+F 6 "Value" H 5100 3750 60  0001 C CNN "ConradPN"
+	1    5100 3750
+	-1   0    0    1
+$EndComp
+Wire Wire Line
+	5300 3750 5500 3750
+Connection ~ 5500 3750
 $EndSCHEMATC

Commit message: Updated the schematic for the BOM and generated the BOM
Parts:
- U101: ConradPN (none) -> 1262416 - 62; Link (none) -> Value; MPN (none) -> LP2980IM5-3.0/NOPB
Changed lines of the file:
@@
 F 2 "Housings_SOT-23_SOT-143_TSOT-6:SOT-23-5" H 3400 1850 60  0001 C CNN
 F 3 "" H 3400 1850 60  0000 C CNN
+F 4 "LP2980IM5-3.0/NOPB" H 3400 1850 60  0001 C CNN "MPN"
+F 5 "Value" H 3400 1850 60  0001 C CNN "Link"
+F 6 "1262416 - 62" H 3400 1850 60  0001 C CNN "ConradPN"
 	1    3400 1850
 	1    0    0    -1

Commit message: Checkin before moving to Vagrant
Parts:
- added R? (x4): 10K, symbol R
Connections:
- wire segments 37 -> 46
Changed lines of the file:
@@
 LIBS:valves
 LIBS:DasBlinkInput
-LIBS:DasBlinkInput-cache
 EELAYER 25 0
 EELAYER END
@@
 L CONN_01X05 P105
 U 1 1 5561D7BD
-P 8650 1800
-F 0 "P105" H 8650 2100 50  0000 C CNN
-F 1 "Output" V 8750 1800 50  0000 C CNN
-F 2 "Pin_Headers:Pin_Header_Straight_1x05" H 8650 1800 60  0001 C CNN
-F 3 "" H 8650 1800 60  0000 C CNN
-F 4 "Value" H 8650 1800 60  0001 C CNN "MPN"
-F 5 "Value" H 8650 1800 60  0001 C CNN "ConradPN"
-	1    8650 1800
+P 9100 1800
+F 0 "P105" H 9100 2100 50  0000 C CNN
+F 1 "Output" V 9200 1800 50  0000 C CNN
+F 2 "Pin_Headers:Pin_Header_Straight_1x05" H 9100 1800 60  0001 C CNN
+F 3 "" H 9100 1800 60  0000 C CNN
+F 4 "Value" H 9100 1800 60  0001 C CNN "MPN"
+F 5 "Value" H 9100 1800 60  0001 C CNN "ConradPN"
+	1    9100 1800
 	1    0    0    -1
 $EndComp
@@
 L C C101
 U 1 1 5561E2B3
-P 2050 2350
-F 0 "C101" H 2075 2450 50  0000 L CNN
-F 1 "1U" H 2075 2250 50  0000 L CNN
-F 2 "Capacitors_SMD:C_0805_HandSoldering" H 2088 2200 30  0001 C CNN
-F 3 "" H 2050 2350 60  0000 C CNN
-	1    2050 2350
+P 1850 2350
+F 0 "C101" H 1875 2450 50  0000 L CNN
+F 1 "1U" H 1875 2250 50  0000 L CNN
+F 2 "Capacitors_SMD:C_0805_HandSoldering" H 1888 2200 30  0001 C CNN
+F 3 "" H 1850 2350 60  0000 C CNN
+	1    1850 2350
 	1    0    0    -1
 $EndComp
@@
 Connection ~ 5500 4450
 Wire Wire Line
-	8450 1600 6700 1600
-Wire Wire Line
-	8450 1700 7450 1700
+	6700 1600 8900 1600
+Wire Wire Line
+	7450 1700 8900 1700
 Wire Wire Line
 	7450 1700 7450 2900
@@
 	7450 2900 6700 2900
 Wire Wire Line
-	8450 1800 7600 1800
+	7600 1800 8900 1800
 Wire Wire Line
 	7600 1800 7600 4050
@@
 	7600 4050 6700 4050
 Wire Wire Line
-	8450 1900 7700 1900
+	7700 1900 8900 1900
 Wire Wire Line
 	7700 1900 7700 5250
@@
 	7700 5250 6750 5250
 Wire Wire Line
-	8450 2000 8250 2000
+	8900 2000 8250 2000
 Wire Wire Line
 	8250 2000 8250 2450
@@
 	1150 1550 2600 1550
 Wire Wire Line
-	2050 2200 2050 1550
-Connection ~ 2050 1550
-Wire Wire Line
-	2050 2500 2050 3050
-Wire Wire Line
-	2050 3050 4400 3050
+	1850 1550 1850 2200
+Connection ~ 1850 1550
+Wire Wire Line
+	1850 2500 1850 3050
+Wire Wire Line
+	1850 3050 4400 3050
 Wire Wire Line
 	3400 2550 3400 3300
@@
 L R R103
 U 1 1 5561E72D
-P 2400 2350
-F 0 "R103" V 2480 2350 50  0000 C CNN
-F 1 "0" V 2400 2350 50  0000 C CNN
-F 2 "Resistors_SMD:R_0805_HandSoldering" V 2330 2350 30  0001 C CNN
-F 3 "" H 2400 2350 30  0000 C CNN
-	1    2400 2350
-	1    0    0    -1
+P 2250 1750
+F 0 "R103" V 2330 1750 50  0000 C CNN
+F 1 "0" V 2250 1750 50  0000 C CNN
+F 2 "Resistors_SMD:R_0805_HandSoldering" V 2180 1750 30  0001 C CNN
+F 3 "" H 2250 1750 30  0000 C CNN
+	1    2250 1750
+	0    1    1    0
 $EndComp
 Wire Wire Line
 	2600 1750 2400 1750
-Wire Wire Line
-	2400 1750 2400 2200
-Wire Wire Line
-	2400 2500 2400 3050
-Connection ~ 2400 3050
 NoConn ~ 2600 2050
 Text GLabel 4750 1550 2    60   Input ~ 0
@@
 	5300 3750 5500 3750
 Connection ~ 5500 3750
+$Comp
+L R R?
+U 1 1 55A0F5AF
+P 8050 1200
+F 0 "R?" V 8130 1200 50  0000 C CNN
+F 1 "10K" V 8050 1200 50  0000 C CNN
+F 2 "" V 7980 1200 30  0000 C CNN
+F 3 "" H 8050 1200 30  0000 C CNN
+	1    8050 1200
+	1    0    0    -1
+$EndComp
+$Comp
+L R R?
+U 1 1 55A0F734
+P 8300 1200
+F 0 "R?" V 8380 1200 50  0000 C CNN
+F 1 "10K" V 8300 1200 50  0000 C CNN
+F 2 "" V 8230 1200 30  0000 C CNN
+F 3 "" H 8300 1200 30  0000 C CNN
+	1    8300 1200
+	1    0    0    -1
+$EndComp
+$Comp
+L R R?
+U 1 1 55A0F7B4
+P 8550 1200
+F 0 "R?" V 8630 1200 50  0000 C CNN
+F 1 "10K" V 8550 1200 50  0000 C CNN
+F 2 "" V 8480 1200 30  0000 C CNN
+F 3 "" H 8550 1200 30  0000 C CNN
+	1    8550 1200
+	1    0    0    -1
+$EndComp
+$Comp
+L R R?
+U 1 1 55A0F825
+P 8800 1200
+F 0 "R?" V 8880 1200 50  0000 C CNN
+F 1 "10K" V 8800 1200 50  0000 C CNN
+F 2 "" V 8730 1200 30  0000 C CNN
+F 3 "" H 8800 1200 30  0000 C CNN
+	1    8800 1200
+	1    0    0    -1
+$EndComp
+Wire Wire Line
+	8050 1350 8050 1600
+Connection ~ 8050 1600
+Wire Wire Line
+	8300 1350 8300 1700
+Connection ~ 8300 1700
+Wire Wire Line
+	8550 1350 8550 1800
+Connection ~ 8550 1800
+Wire Wire Line
+	8800 1350 8800 1900
+Connection ~ 8800 1900
+Text GLabel 7500 900  0    60   Input ~ 0
+3V
+Wire Wire Line
+	7500 900  8800 900
+Wire Wire Line
+	8800 900  8800 1050
+Wire Wire Line
+	8550 900  8550 1050
+Connection ~ 8550 900
+Wire Wire Line
+	8300 900  8300 1050
+Connection ~ 8300 900
+Wire Wire Line
+	8050 900  8050 1050
+Connection ~ 8050 900
+Wire Wire Line
+	2100 1750 2000 1750
+Wire Wire Line
+	2000 1750 2000 1550
+Connection ~ 2000 1550
 $EndSCHEMATC

Commit message: Clean up and correctsion to the layout. Added the pull up resistors
Parts:
- C101, C102: footprint Capacitors_SMD:C_0805_HandSoldering -> Capacitors_SMD:C_0805
- R101, R102, R103: footprint Resistors_SMD:R_0805_HandSoldering -> Resistors_SMD:R_0805
- R104, R105, R106, R107: renamed from R?; footprint (none) -> Resistors_SMD:R_0805
Changed lines of the file:
@@
 LIBS:valves
 LIBS:DasBlinkInput
+LIBS:DasBlinkInput-cache
 EELAYER 25 0
 EELAYER END
@@
 F 0 "C101" H 1875 2450 50  0000 L CNN
 F 1 "1U" H 1875 2250 50  0000 L CNN
-F 2 "Capacitors_SMD:C_0805_HandSoldering" H 1888 2200 30  0001 C CNN
+F 2 "Capacitors_SMD:C_0805" H 1888 2200 30  0001 C CNN
 F 3 "" H 1850 2350 60  0000 C CNN
 	1    1850 2350
@@
 F 0 "C102" H 4425 2600 50  0000 L CNN
 F 1 "1U" H 4425 2400 50  0000 L CNN
-F 2 "Capacitors_SMD:C_0805_HandSoldering" H 4438 2350 30  0001 C CNN
+F 2 "Capacitors_SMD:C_0805" H 4438 2350 30  0001 C CNN
 F 3 "" H 4400 2500 60  0000 C CNN
 	1    4400 2500
@@
 F 0 "R103" V 2330 1750 50  0000 C CNN
 F 1 "0" V 2250 1750 50  0000 C CNN
-F 2 "Resistors_SMD:R_0805_HandSoldering" V 2180 1750 30  0001 C CNN
+F 2 "Resistors_SMD:R_0805" V 2180 1750 30  0001 C CNN
 F 3 "" H 2250 1750 30  0000 C CNN
 	1    2250 1750
@@
 F 0 "R101" V 1330 3750 50  0000 C CNN
 F 1 "10K" V 1250 3750 50  0000 C CNN
-F 2 "Resistors_SMD:R_0805_HandSoldering" V 1180 3750 30  0001 C CNN
+F 2 "Resistors_SMD:R_0805" V 1180 3750 30  0001 C CNN
 F 3 "" H 1250 3750 30  0000 C CNN
 	1    1250 3750
@@
 F 0 "R102" V 1330 4450 50  0000 C CNN
 F 1 "10K" V 1250 4450 50  0000 C CNN
-F 2 "Resistors_SMD:R_0805_HandSoldering" V 1180 4450 30  0001 C CNN
+F 2 "Resistors_SMD:R_0805" V 1180 4450 30  0001 C CNN
 F 3 "" H 1250 4450 30  0000 C CNN
 	1    1250 4450
@@
 Connection ~ 5500 3750
 $Comp
-L R R?
+L R R104
 U 1 1 55A0F5AF
 P 8050 1200
-F 0 "R?" V 8130 1200 50  0000 C CNN
+F 0 "R104" V 8130 1200 50  0000 C CNN
 F 1 "10K" V 8050 1200 50  0000 C CNN
-F 2 "" V 7980 1200 30  0000 C CNN
+F 2 "Resistors_SMD:R_0805" V 7980 1200 30  0001 C CNN
 F 3 "" H 8050 1200 30  0000 C CNN
 	1    8050 1200
@@
 $EndComp
 $Comp
-L R R?
+L R R105
 U 1 1 55A0F734
 P 8300 1200
-F 0 "R?" V 8380 1200 50  0000 C CNN
+F 0 "R105" V 8380 1200 50  0000 C CNN
 F 1 "10K" V 8300 1200 50  0000 C CNN
-F 2 "" V 8230 1200 30  0000 C CNN
+F 2 "Resistors_SMD:R_0805" V 8230 1200 30  0001 C CNN
 F 3 "" H 8300 1200 30  0000 C CNN
 	1    8300 1200
@@
 $EndComp
 $Comp
-L R R?
+L R R106
 U 1 1 55A0F7B4
 P 8550 1200
-F 0 "R?" V 8630 1200 50  0000 C CNN
+F 0 "R106" V 8630 1200 50  0000 C CNN
 F 1 "10K" V 8550 1200 50  0000 C CNN
-F 2 "" V 8480 1200 30  0000 C CNN
+F 2 "Resistors_SMD:R_0805" V 8480 1200 30  0001 C CNN
 F 3 "" H 8550 1200 30  0000 C CNN
 	1    8550 1200
@@
 $EndComp
 $Comp
-L R R?
+L R R107
 U 1 1 55A0F825
 P 8800 1200
-F 0 "R?" V 8880 1200 50  0000 C CNN
+F 0 "R107" V 8880 1200 50  0000 C CNN
 F 1 "10K" V 8800 1200 50  0000 C CNN
-F 2 "" V 8730 1200 30  0000 C CNN
+F 2 "Resistors_SMD:R_0805" V 8730 1200 30  0001 C CNN
 F 3 "" H 8800 1200 30  0000 C CNN
 	1    8800 1200
